File: DGD05473.kicad_sch (KiCad schematic)
At the start: 43 parts, among them Q1 DMN6017SK3, Q2 DMN6017SK3, Q3 DMN6017SK3, Q4 DMN6017SK3, U1 dgd05473, U10 C2012X7S2A105K125AE_p, U11 C2012NP02A102J060AA_p, U12 C2012NP02A102J060AA_p, U13 C2012X7S2A105K125AE_p, U15 CAA573X7S2A476M640LH_p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

Commit message: Add files via upload
Parts:
- U8: value C2012X7S2A105K125AE_p -> ATLI_860080772001_10uF
- renumbered V3 to V1, V4 to V2, V5 to V3, V6 to V4, V1 to V5, V2 to V6
Changed lines of the file:
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@@
 	(title_block
 		(title "HIGH-FREQUENCY HIGH-SIDE AND LOW-SIDE GATE DRIVER")
-		(date "2025-04-14")
+		(date "2025-04-19")
 		(rev "1")
 		(company "astroelectronic@")
@@
 		(dnp no)
 		(fields_autoplaced yes)
-		(property "Reference" "V6"
+		(property "Reference" "V4"
 			(at 54.61 133.2201 0)
 			(effects
@@
 			(project "DGD05473"
 				(path "/79bac4d6-c0b7-44a0-a7ef-b66f4209da8b"
-					(reference "V6")
+					(reference "V4")
 					(unit 1)
 				)
@@
 		(dnp no)
 		(fields_autoplaced yes)
-		(property "Reference" "V4"
+		(property "Reference" "V2"
 			(at 54.61 57.0201 0)
 			(effects
@@
 			(project "DGD05473"
 				(path "/79bac4d6-c0b7-44a0-a7ef-b66f4209da8b"
-					(reference "V4")
+					(reference "V2")
 					(unit 1)
 				)
@@
 		(dnp no)
 		(fields_autoplaced yes)
-		(property "Reference" "V5"
+		(property "Reference" "V3"
 			(at 41.91 145.9201 0)
 			(effects
@@
 			(project "DGD05473"
 				(path "/79bac4d6-c0b7-44a0-a7ef-b66f4209da8b"
-					(reference "V5")
+					(reference "V3")
 					(unit 1)
 				)
@@
 			)
 		)
-		(property "Value" "C2012X7S2A105K125AE_p"
+		(property "Value" "ATLI_860080772001_10uF"
 			(at 257.81 33.0199 0)
 			(effects
@@
 			)
 		)
-		(property "Sim.Library" "c2012x7s2a105k125ae_p.mod"
+		(property "Sim.Library" "ATLI_860080772001_10uF.lib"
 			(at 254 31.75 0)
 			(effects
@@
 			)
 		)
-		(property "Sim.Name" "C2012X7S2A105K125AE_p"
+		(property "Sim.Name" "ATLI_860080772001_10uF"
 			(at 254 31.75 0)
 			(effects
@@
 			)
 		)
-		(property "Sim.Pins" "1=n1 2=n2"
+		(property "Sim.Pins" "1=1 2=2"
 			(at 254 31.75 0)
 			(effects
@@
 		(dnp no)
 		(fields_autoplaced yes)
-		(property "Reference" "V1"
+		(property "Reference" "V5"
 			(at 105.41 176.4001 0)
 			(effects
@@
 			(project ""
 				(path "/79bac4d6-c0b7-44a0-a7ef-b66f4209da8b"
-					(reference "V1")
+					(reference "V5")
 					(unit 1)
 				)
@@
 		(dnp no)
 		(fields_autoplaced yes)
-		(property "Reference" "V2"
+		(property "Reference" "V6"
 			(at 118.11 176.4001 0)
 			(effects
@@
 			(project "DGD05473"
 				(path "/79bac4d6-c0b7-44a0-a7ef-b66f4209da8b"
-					(reference "V2")
+					(reference "V6")
 					(unit 1)
 				)
@@
 		(dnp no)
 		(fields_autoplaced yes)
-		(property "Reference" "V3"
+		(property "Reference" "V1"
 			(at 41.91 69.7201 0)
 			(effects
@@
 			(project "DGD05473"
 				(path "/79bac4d6-c0b7-44a0-a7ef-b66f4209da8b"
-					(reference "V3")
+					(reference "V1")
 					(unit 1)
 				)
